Commit message: Looks like TF tree is now more correct- base_footprint is a child of base_link. Parts of robot are no longer detached, but costmaps are still displaced.

File: pmb2_description/urdf/base/base.urdf.xacro (robot description, xacro)
@@ -65,6 +65,8 @@
     <joint name="${name}_footprint_joint" type="fixed">
       <origin xyz="0 0 ${wheel_radius}" rpy="0 0 0" />
-      <child link="${name}_link" />
-      <parent link="${name}_footprint"/>
+      <!--child link="${name}_link" />
+      <parent link="${name}_footprint"/--> <!-- AE: 06 Nov 2023 -->
+      <child link="${name}_footprint" />
+      <parent link="${name}_link"/>
     </joint>
   <!-- gazebo parameters are given here for base_link thru base_footprint -->
